Commit message: add fictitious urdf frames to peg/hole for tf frame computations. decrease friction from 1.0 to 0.2 of peg to ease peg insertion task.

File: franka_description/robots/hole.urdf (robot description, URDF)
Before this commit: robot hole, 1 links, 0 joints
Links:
- removed link hole_link
- added link hole_base_link, mass 1; collision box size=0.01193474204277948 0.0165 0.12; collision box size=0.01193474204277948 0.0165 0.12
- added link hole_root_link
- added link hole_top_link
Joints:
- added joint hole_root_joint: type fixed, parent hole_root_link, child hole_base_link, origin xyz=0 0 0 rpy=0 0 0
- added joint hole_top_joint: type fixed, parent hole_root_link, child hole_top_link, origin xyz=0 0 0.12 rpy=0 0 0

File: franka_description/robots/panda_arm_peg.urdf.xacro (robot description, xacro)
@@ -6,6 +6,6 @@
   <xacro:arg name="peg" default="false"/> <!-- Should a peg be mounted at the flange?" -->
   <xacro:property name="arm_id" value="$(arg arm_id)" />
+  <!-- Create a URDF for a real hardware -->
   <xacro:unless value="$(arg gazebo)">
-    <!-- Create a URDF for a real hardware -->
     <xacro:include filename="$(find franka_description)/robots/panda_arm.xacro" />
     <xacro:panda_arm arm_id="${arm_id}" safety_distance="0.03"/>
@@ -19,4 +19,5 @@
     </xacro:if>
   </xacro:unless>
+  <!-- Separate URDF for simulation... -->
   <xacro:if value="$(arg gazebo)">
     <xacro:arg name="xyz" default="0 0 0" />

File: franka_description/robots/panda_gazebo.xacro (robot description, xacro)
@@ -378,4 +378,16 @@
       </inertial>
 	  </link>
+    <gazebo reference="${ns}_peg">
+      <mu1>0.2</mu1>
+      <mu2>0.2</mu2>
+    </gazebo>
+    <!-- add a dummy link to the tip of the peg for rviz/kdl purposes -->
+    <joint name="${ns}_tip_joint" type="fixed">
+        <parent link="${ns}_peg"/>
+        <child link="${ns}_tip"/>
+        <origin xyz="0 0 0.111" rpy="0 0 0"/>
+    </joint>
+    <link name="${ns}_tip">
+    </link>
   </xacro:macro>
 </robot>

File: franka_description/robots/peg.xacro (robot description, xacro)
@@ -17,5 +17,4 @@
     <!-- <xacro:property name="mass" value="5.0" /> -->
     <link name="${ns}_peg">
-      <!-- <origin xyz="0 0 0" rpy="0 0 0"/> -->
       <visual>
         <origin xyz="0 0 ${length/2}" rpy="0 0 0"/>
@@ -39,4 +38,12 @@
       </inertial>
 	  </link>
+    <!-- add a dummy link to the tip of the peg for rviz/kdl purposes -->
+    <joint name="${ns}_tip_joint" type="fixed">
+        <parent link="${ns}_peg"/>
+        <child link="${ns}_tip"/>
+        <origin xyz="0 0 0.111" rpy="0 0 0"/>
+    </joint>
+    <link name="${ns}_tip">
+    </link>
   </xacro:macro>
 </robot>
