Commit message: change root link to be top of the hole flush with surface

File: franka_description/robots/holerootbase.urdf (robot description, URDF)
Before this commit: robot hole, 3 links, 2 joints
Joints:
- joint hole_root_joint: origin xyz=0 0 -0.12 rpy=0 0 0 -> xyz=0 0 0 rpy=0 0 0
- joint hole_top_joint: origin xyz=0 0 0 rpy=0 0 0 -> xyz=0 0 0.12 rpy=0 0 0
