Commit message: Add sphere urdf. Fix peg urdf.

File: franka_description/robots/panda_arm_sphere.xacro (robot description, xacro)
@@ -4,5 +4,5 @@
   <xacro:arg name="hand"   default="false" /> <!-- Should a franka_gripper be mounted at the flange?" -->
   <xacro:arg name="gazebo" default="false" /> <!-- Is the robot being simulated in gazebo?" -->
-  <xacro:arg name="peg" default="true"/> <!-- Should a peg be mounted at the flange?" -->
+  <xacro:arg name="sphere" default="false"/> <!-- Should a sphere be mounted at the flange?" -->
   <xacro:property name="arm_id" value="$(arg arm_id)" />
   <!-- Create a URDF for a real hardware -->
@@ -14,7 +14,7 @@
       <xacro:hand ns="${arm_id}" rpy="0 0 ${-pi/4}" connected_to="${arm_id}_link8" safety_distance="0.03"/>
     </xacro:if>
-    <xacro:if value="$(arg peg)">
-      <xacro:include filename="$(find franka_description)/robots/peg.xacro"/>
-      <xacro:peg ns="${arm_id}" rpy="0 0 ${-pi/4}" connected_to="${arm_id}_link8"/>
+    <xacro:if value="$(arg sphere)">
+      <xacro:include filename="$(find franka_description)/robots/sphere.xacro"/>
+      <xacro:sphere ns="${arm_id}" rpy="0 0 ${-pi/4}" connected_to="${arm_id}_link8"/>
     </xacro:if>
   </xacro:unless>
@@ -32,6 +32,6 @@
       <xacro:gazebo-joint joint="${arm_id}_finger_joint2" transmission="hardware_interface/EffortJointInterface" />
     </xacro:if>
-    <xacro:if value="$(arg peg)">
-      <xacro:peg ns="${arm_id}" rpy="0 0 ${-pi/4}" connected_to="${arm_id}_link8" />
+    <xacro:if value="$(arg sphere)">
+      <xacro:sphere ns="${arm_id}" rpy="0 0 ${-pi/4}" connected_to="${arm_id}_link8" />
     </xacro:if>
     <!-- Gazebo requires a joint to a link called "world" for statically mounted robots -->

File: franka_description/robots/peg.xacro (robot description, xacro)
@@ -2,5 +2,5 @@
 <robot xmlns:xacro="http://www.ros.org/wiki/xacro" name="peg">
   <!-- utils /-->
-  <xacro:include filename="$(find franka_panda_description)/robots/utils.xacro"/>
+  <xacro:include filename="$(find franka_description)/robots/utils.xacro"/>
   <xacro:macro name="peg" params="connected_to:='' ns:='' rpy:='0 0 0' xyz:='0 0 0' ">
     <xacro:unless value="${connected_to == ''}">

File: franka_description/robots/utils.xacro (robot description, xacro)
@@ -119,3 +119,9 @@
              ixy="0" iyz="0" ixz="0"/>
   </xacro:macro>
+  <xacro: macro name="sphere_intertia_def" params="radius mass">
+    <inertia ixx="${2 * mass * radius * radius / 5}"
+             iyy="${2 * mass * radius * radius / 5}"
+             izz="${2 * mass * radius * radius / 5}"
+             ixy="0" iyz="0" ixz="0"/>
+  </xacro:macro>
 </robot>
