Commit message: Remove whitespace

File: franka_description/robots/utils.xacro (robot description, xacro)
@@ -119,5 +119,5 @@
              ixy="0" iyz="0" ixz="0"/>
   </xacro:macro>
-  <xacro: macro name="sphere_intertia_def" params="radius mass">
+  <xacro:macro name="sphere_inertia_def" params="radius mass">
     <inertia ixx="${2 * mass * radius * radius / 5}"
              iyy="${2 * mass * radius * radius / 5}"
