Commit message: Add tip link

File: franka_description/robots/sphere.xacro (robot description, xacro)
@@ -2,6 +2,6 @@
 <robot xmlns:xacro="http://www.ros.org/wiki/xacro" name="sphere">
   <!-- utils /-->
-  <xacro:include filename="$(find franka_panda_description)/robots/utils.xacro"/>
-  <xacro:macro name="sphere" params="connected_to:='' ns:='' rpy:='0 0 0' xyz:='0 0 0' ">
+  <xacro:include filename="$(find franka_description)/robots/utils.xacro"/>
+  <xacro:macro name="sphere_shape" params="connected_to:='' ns:='' rpy:='0 0 0' xyz:='0 0 0' ">
     <xacro:unless value="${connected_to == ''}">
       <joint name="${ns}_sphere_joint" type="fixed">
@@ -39,5 +39,5 @@
         <parent link="${ns}_peg"/>
         <child link="${ns}_tip"/>
-        <origin xyz="0 0 0.555" rpy="0 0 0"/>
+        <origin xyz="0 0 0.111" rpy="0 0 0"/>
     </joint>
     <link name="${ns}_tip">

Commit message: Fix name from peg to sphere

File: franka_description/robots/sphere.xacro (robot description, xacro)
@@ -37,7 +37,7 @@
     <!-- add a dummy link to the tip of the peg for rviz/kdl purposes -->
     <joint name="${ns}_tip_joint" type="fixed">
-        <parent link="${ns}_peg"/>
+        <parent link="${ns}_sphere"/>
         <child link="${ns}_tip"/>
-        <origin xyz="0 0 0.111" rpy="0 0 0"/>
+        <origin xyz="0 0 0.555" rpy="0 0 0"/>
     </joint>
     <link name="${ns}_tip">

Commit message: update tip frame to match diameter

File: franka_description/robots/sphere.xacro (robot description, xacro)
@@ -39,5 +39,5 @@
         <parent link="${ns}_sphere"/>
         <child link="${ns}_tip"/>
-        <origin xyz="0 0 ${radius}" rpy="0 0 0"/>
+        <origin xyz="0 0 $(0.785398163397 - {radius})" rpy="0 0 0"/>
     </joint>
     <link name="${ns}_tip">
