Commit message: fix some launch params to use arm_id instead of ns for 0.9.0. add collision bitmasks to various sim models for contact project. edit the joint impedance example controller to print the custom state and diagnostic

File: franka_description/robots/panda_attachments.urdf.xacro (robot description, xacro)
@@ -13,5 +13,5 @@
     <xacro:if value="$(arg hand)">
       <xacro:include filename="$(find franka_description)/robots/hand.xacro"/>
-      <xacro:hand ns="${arm_id}" rpy="0 0 ${-pi/4}" connected_to="${arm_id}_link8" safety_distance="0.03"/>
+      <xacro:hand arm_id="${arm_id}" rpy="0 0 ${-pi/4}" connected_to="${arm_id}_link8" safety_distance="0.03"/>
     </xacro:if>
     <xacro:if value="$(arg peg)">
@@ -33,5 +33,5 @@
     <xacro:panda_arm arm_id="${arm_id}" />
     <xacro:if value="$(arg hand)">
-      <xacro:hand ns="${arm_id}" rpy="0 0 ${-pi/4}" connected_to="${arm_id}_link8" />
+      <xacro:hand arm_id="${arm_id}" rpy="0 0 ${-pi/4}" connected_to="${arm_id}_link8" />
       <xacro:gazebo-joint joint="${arm_id}_finger_joint1" transmission="hardware_interface/EffortJointInterface" />
       <xacro:gazebo-joint joint="${arm_id}_finger_joint2" transmission="hardware_interface/EffortJointInterface" />

File: franka_description/robots/panda_gazebo.xacro (robot description, xacro)
@@ -40,13 +40,5 @@
       </inertial>
     </link>
-    <gazebo reference="${arm_id}_link0">
-      <collision>
-        <surface>
-          <contact>
-            <collide_bitmask>0x0</collide_bitmask>
-          </contact>
-        </surface>
-      </collision>
-    </gazebo>
+    <xacro:gazebo-coll-bitmask link="${arm_id}_link0" bitmask="0x0" />
     <link name="${arm_id}_link1">
       <visual>
@@ -220,13 +212,5 @@
       </inertial>
     </link>
-    <gazebo reference="${arm_id}_link6">
-      <collision>
-        <surface>
-          <contact>
-            <collide_bitmask>0x001</collide_bitmask>
-          </contact>
-        </surface>
-      </collision>
-    </gazebo>
+    <xacro:gazebo-coll-bitmask link="${arm_id}_link6" bitmask="0x01" />
     <joint name="${arm_id}_joint6" type="revolute">
       <safety_controller k_position="100.0" k_velocity="40.0" soft_lower_limit="-0.0175" soft_upper_limit="3.7525"/>
@@ -259,13 +243,5 @@
       </inertial>
     </link>
-    <gazebo reference="${arm_id}_link7">
-      <collision>
-        <surface>
-          <contact>
-            <collide_bitmask>0x01</collide_bitmask>
-          </contact>
-        </surface>
-      </collision>
-    </gazebo>
+    <xacro:gazebo-coll-bitmask link="${arm_id}_link7" bitmask="0x01" />
     <joint name="${arm_id}_joint7" type="revolute">
       <safety_controller k_position="100.0" k_velocity="40.0" soft_lower_limit="-2.8973" soft_upper_limit="2.8973"/>
@@ -313,4 +289,5 @@
       </inertial>
     </link>
+    <xacro:gazebo-coll-bitmask link="${arm_id}_hand" bitmask="0x01" />
     <xacro:macro name="finger-collision" params="sign">
       <!-- screw mount -->
@@ -366,4 +343,6 @@
     <xacro:gazebo-friction link="${arm_id}_leftfinger" mu="1.13" />
     <xacro:gazebo-friction link="${arm_id}_rightfinger" mu="1.13" />
+    <xacro:gazebo-coll-bitmask link="${arm_id}_leftfinger" bitmask="0x01" />
+    <xacro:gazebo-coll-bitmask link="${arm_id}_rightfinger" bitmask="0x01" />
     <joint name="${arm_id}_finger_joint1" type="prismatic">
       <parent link="${arm_id}_hand"/>
@@ -478,5 +457,5 @@
     </joint>
     <link name="${ns}_tip">
-    </link>1
+    </link>
   </xacro:macro>
 </robot>

File: franka_description/robots/utils.xacro (robot description, xacro)
@@ -43,4 +43,15 @@
           </friction>
           <bounce/>
+        </surface>
+      </collision>
+    </gazebo>
+  </xacro:macro>
+  <xacro:macro name="gazebo-coll-bitmask" params="link bitmask">
+    <gazebo reference="${link}">
+      <collision>
+        <surface>
+          <contact>
+            <collide_bitmask>${bitmask}</collide_bitmask>
+          </contact>
         </surface>
       </collision>
@@ -107,7 +118,7 @@
   <!-- Little helper macro to define the inertia matrix needed for links. -->
   <xacro:macro name="cuboid_inertia_def" params="width height length mass">
-    <inertia ixx="${mass * (height * height + length * length) / 12}"
-             iyy="${mass * (width * width + length * length) / 12}"
-             izz="${mass * (width * width + height * height) / 12}"
+    <inertia ixx="${mass * (height * height + width * width) / 12}"
+             iyy="${mass * (height * height + length * length) / 12}"
+             izz="${mass * (width * width + length * length) / 12}"
              ixy="0" iyz="0" ixz="0"/>
   </xacro:macro>
