Commit message: add peg model to urdf model/sim. Strange issue with what I believe is grav comp overcompensating and causing arm to shoot up. Happens without the peg as well so this is seemingly not caused by the addition of peg model?

File: franka_description/robots/panda_gazebo.xacro (robot description, xacro)
@@ -342,3 +342,41 @@
     </joint>
   </xacro:macro>
+  <xacro:macro name="peg" params="connected_to:='' ns:='' xyz:='0 0 0' rpy:='0 0 0'">
+    <xacro:include filename="$(find franka_description)/robots/utils.xacro"/>
+    <xacro:unless value="${connected_to == ''}">
+      <joint name="${ns}_peg_joint" type="fixed">
+        <parent link="${connected_to}"/>
+        <child link="${ns}_peg"/>
+        <origin xyz="${xyz}" rpy="${rpy}"/>
+      </joint>
+    </xacro:unless>
+     <!-- 1" diameter and 4.375" length (including mount plate) -->
+    <xacro:property name="radius" value="0.0127" />
+    <xacro:property name="length" value="0.111125" />
+    <xacro:property name="mass" value="0.23" />
+    <!-- <xacro:property name="mass" value="5.0" /> -->
+    <link name="${ns}_peg">
+      <!-- <origin xyz="0 0 0" rpy="0 0 0"/> -->
+      <visual>
+        <origin xyz="0 0 ${length/2}" rpy="0 0 0"/>
+        <geometry>
+          <cylinder length="${length}" radius="${radius}"/>
+        </geometry>
+        <material name="gray">
+          <color rgba="0.75 0.75 0.75 1"/>
+        </material>
+      </visual>
+      <collision>
+        <origin xyz="0 0 ${length/2}" rpy="0 0 0"/>
+        <geometry>
+          <cylinder length="${length}" radius="${radius}"/>
+        </geometry>
+      </collision>
+      <inertial>
+        <origin xyz="0 0 ${length/2}"/>
+        <mass value="${mass}"/>
+      	<cylinder_inertia_def radius="${radius}" length="${length}" mass="${mass}"/>
+      </inertial>
+	  </link>
+  </xacro:macro>
 </robot>

File: franka_description/robots/utils.xacro (robot description, xacro)
@@ -103,3 +103,19 @@
     </inertial>
   </xacro:macro>
+  <!-- taken from https://github.com/epfl-lasa/kuka-lwr-ros/blob/2533aa1bb521d531845cea45c93a4ded1ccf6539/kuka_lwr/lwr_description/model/utils.xacro -->
+  <xacro:property name="M_PI" value="3.1415926535897931"/>
+  <!-- Little helper macro to define the inertia matrix needed for links. -->
+  <xacro:macro name="cuboid_inertia_def" params="width height length mass">
+    <inertia ixx="${mass * (height * height + length * length) / 12}"
+             iyy="${mass * (width * width + length * length) / 12}"
+             izz="${mass * (width * width + height * height) / 12}"
+             ixy="0" iyz="0" ixz="0"/>
+  </xacro:macro>
+  <!-- length is along the z-axis! -->
+  <xacro:macro name="cylinder_inertia_def" params="radius length mass">
+    <inertia ixx="${mass * (3 * radius * radius + length * length) / 12}"
+             iyy="${mass * (3 * radius * radius + length * length) / 12}"
+             izz="${mass * radius* radius / 2}"
+             ixy="0" iyz="0" ixz="0"/>
+  </xacro:macro>
 </robot>

Commit message: fix EE overcompensation problem. Add dyn reconfigure of pose gains in interactive marker script

File: franka_description/robots/panda_gazebo.xacro (robot description, xacro)
@@ -355,5 +355,4 @@
     <xacro:property name="length" value="0.111125" />
     <xacro:property name="mass" value="0.23" />
-    <!-- <xacro:property name="mass" value="5.0" /> -->
     <link name="${ns}_peg">
       <!-- <origin xyz="0 0 0" rpy="0 0 0"/> -->

Commit message: Add sphere to panda_gazebo.xacro

File: franka_description/robots/panda_gazebo.xacro (robot description, xacro)
@@ -391,3 +391,48 @@
     </link>
   </xacro:macro>
+   <xacro:macro name="sphere_shape" params="connected_to:='' ns:='' rpy:='0 0 0' xyz:='0 0 0' ">
+    <xacro:unless value="${connected_to == ''}">
+      <joint name="${ns}_sphere_joint" type="fixed">
+        <parent link="${connected_to}"/>
+        <child link="${ns}_sphere"/>
+        <origin xyz="${xyz}" rpy="${rpy}"/>
+      </joint>
+    </xacro:unless>
+    <xacro:property name="radius" value="0.0555625" />
+    <xacro:property name="mass" value="0.23" />
+    <link name="${ns}_sphere">
+      <visual>
+        <origin xyz="0 0 ${radius}" rpy="0 0 0"/>
+        <geometry>
+          <sphere radius="${radius}"/>
+        </geometry>
+        <material name="gray">
+          <color rgba="0.75 0.75 0.75 1"/>
+        </material>
+      </visual>
+      <collision>
+        <origin xyz="0 0 ${radius}" rpy="0 0 0"/>
+        <geometry>
+          <sphere radius="${radius}"/>
+        </geometry>
+      </collision>
+      <inertial>
+        <origin xyz="0 0 ${radius}"/>
+        <mass value="${mass}"/>
+      	<sphere_inertia_def radius="${radius}" mass="${mass}"/>
+      </inertial>
+	  </link>
+    <gazebo reference="${ns}_peg">
+      <mu1>0.2</mu1>
+      <mu2>0.2</mu2>
+    </gazebo>
+    <!-- add a dummy link to the tip of the peg for rviz/kdl purposes -->
+    <joint name="${ns}_tip_joint" type="fixed">
+        <parent link="${ns}_peg"/>
+        <child link="${ns}_tip"/>
+        <origin xyz="0 0 0.111" rpy="0 0 0"/>
+    </joint>
+    <link name="${ns}_tip">
+    </link>
+  </xacro:macro>
 </robot>

Commit message: Add sphere

File: franka_description/robots/panda_gazebo.xacro (robot description, xacro)
@@ -423,5 +423,5 @@
       </inertial>
 	  </link>
-    <gazebo reference="${ns}_peg">
+    <gazebo reference="${ns}_sphere">
       <mu1>0.2</mu1>
       <mu2>0.2</mu2>
@@ -429,10 +429,10 @@
     <!-- add a dummy link to the tip of the peg for rviz/kdl purposes -->
     <joint name="${ns}_tip_joint" type="fixed">
-        <parent link="${ns}_peg"/>
+        <parent link="${ns}_sphere"/>
         <child link="${ns}_tip"/>
         <origin xyz="0 0 0.111" rpy="0 0 0"/>
     </joint>
     <link name="${ns}_tip">
-    </link>
+    </link>1
   </xacro:macro>
 </robot>

Commit message: add camera urdf. change robot base collision bitmask to prevent simulation of contacts with the ground

File: franka_description/robots/panda_gazebo.xacro (robot description, xacro)
@@ -33,4 +33,13 @@
       </inertial>
     </link>
+    <gazebo reference="${arm_id}_link0">
+      <collision>
+        <surface>
+          <contact>
+            <collide_bitmask>0x0</collide_bitmask>
+          </contact>
+        </surface>
+      </collision>
+    </gazebo>
     <link name="${arm_id}_link1">
       <visual>

Commit message: Add collision besides bottom link

File: franka_description/robots/panda_gazebo.xacro (robot description, xacro)
@@ -42,5 +42,4 @@
         </geometry>
       </visual>
-      <!--
       <collision>
         <origin rpy="0 0 0" xyz="0 0 0"/>
@@ -49,5 +48,4 @@
         </geometry>
       </collision>
-      -->
       <inertial>
         <origin rpy="0 0 0" xyz="0.003875 0.002081 -0.04762"/>
@@ -74,5 +72,4 @@
         </geometry>
       </visual>
-      <!--
       <collision>
         <origin rpy="0 0 0" xyz="0 0 0"/>
@@ -81,5 +78,4 @@
         </geometry>
       </collision>
-      -->
       <inertial>
         <origin rpy="0 0 0" xyz=" -0.003141 -0.02872  0.003495"/>
@@ -106,5 +102,4 @@
         </geometry>
       </visual>
-      <!--
       <collision>
         <origin rpy="0 0 0" xyz="0 0 0"/>
@@ -113,5 +108,4 @@
         </geometry>
       </collision>
-      -->
       <inertial>
         <origin rpy="0 0 0" xyz="2.7518e-02 3.9252e-02 -6.6502e-02"/>
@@ -138,5 +132,4 @@
         </geometry>
       </visual>
-      <!--
       <collision>
         <origin rpy="0 0 0" xyz="0 0 0"/>
@@ -145,5 +138,4 @@
         </geometry>
       </collision>
-      -->
       <inertial>
         <origin rpy="0 0 0" xyz="-5.317e-02 1.04419e-01 2.7454e-02"/>
@@ -170,5 +162,4 @@
         </geometry>
       </visual>
-      <!--
       <collision>
         <origin rpy="0 0 0" xyz="0 0 0"/>
@@ -177,5 +168,4 @@
         </geometry>
       </collision>
-      -->
       <inertial>
         <origin rpy="0 0 0" xyz="-1.1953e-02 4.1065e-02 -3.8437e-02"/>
@@ -202,5 +192,4 @@
         </geometry>
       </visual>
-      <!--
       <collision>
         <origin rpy="0 0 0" xyz="0 0 0"/>
@@ -209,5 +198,4 @@
         </geometry>
       </collision>
-      -->
       <inertial>
         <origin rpy="0 0 0" xyz="6.0149e-02 -1.4117e-02 -1.0517e-02"/>
@@ -234,5 +222,4 @@
         </geometry>
       </visual>
-      <!--
       <collision>
         <origin rpy="0 0 0" xyz="0 0 0"/>
@@ -241,5 +228,4 @@
         </geometry>
       </collision>
-      -->
       <inertial>
         <origin rpy="0 0 0" xyz="1.0517e-02 -4.252e-03 6.1597e-02"/>
@@ -446,5 +432,5 @@
         <parent link="${ns}_sphere"/>
         <child link="${ns}_tip"/>
-        <origin xyz="0 0 0.111" rpy="0 0 0"/>
+        <origin xyz="0 0 ${radius * 2}" rpy="0 0 0"/>
     </joint>
     <link name="${ns}_tip">

Commit message: up franka state publish rate to 1000 and add bitmask to prevent collisions between last two links and the spawned EE object

File: franka_description/robots/panda_gazebo.xacro (robot description, xacro)
@@ -213,4 +213,13 @@
       </inertial>
     </link>
+    <gazebo reference="${arm_id}_link6">
+      <collision>
+        <surface>
+          <contact>
+            <collide_bitmask>0x001</collide_bitmask>
+          </contact>
+        </surface>
+      </collision>
+    </gazebo>
     <joint name="${arm_id}_joint6" type="revolute">
       <safety_controller k_position="100.0" k_velocity="40.0" soft_lower_limit="-0.0175" soft_upper_limit="3.7525"/>
@@ -243,4 +252,13 @@
       </inertial>
     </link>
+    <gazebo reference="${arm_id}_link7">
+      <collision>
+        <surface>
+          <contact>
+            <collide_bitmask>0x01</collide_bitmask>
+          </contact>
+        </surface>
+      </collision>
+    </gazebo>
     <joint name="${arm_id}_joint7" type="revolute">
       <safety_controller k_position="100.0" k_velocity="40.0" soft_lower_limit="-2.8973" soft_upper_limit="2.8973"/>
@@ -434,5 +452,6 @@
       <mu1 value="${mu}" />
       <mu2 value="${mu}" />
-      <kp>1e5</kp>
+      <!-- previously 1e5 -->
+      <kp>1e4</kp>
       <kd>1e1</kd>
     </gazebo>

File: franka_description/robots/sphere.xacro (robot description, xacro)
@@ -1,3 +1,3 @@
-<?xml version="1.0" encoding="utf-8"?>
+<?xml version="1.0" ?>
 <robot xmlns:xacro="http://www.ros.org/wiki/xacro" name="sphere">
   <!-- utils /-->

Commit message: add eric cousineau's joint friction params to urdf

File: franka_description/robots/panda_gazebo.xacro (robot description, xacro)
@@ -69,5 +69,6 @@
       <axis xyz="0 0 1"/>
       <limit acceleration="15" lower="-2.9671" effort="87" upper="2.9671" velocity="2.5"/>
-      <dynamics D="1" K="7000" mu_coulomb="0" mu_viscous="16" damping="0.003" friction="0.0"/>
+      <!-- <dynamics D="1" K="7000" mu_coulomb="0" mu_viscous="16" damping="0.003" friction="0.0"/> -->
+      <dynamics D="1" K="7000" mu_coulomb="0" mu_viscous="16" damping="0.32" friction="1.045"/>
     </joint>
     <link name="${arm_id}_link2">
@@ -99,5 +100,6 @@
       <axis xyz="0 0 1"/>
       <limit acceleration="7.5" lower="-1.8326" effort="87" upper="1.8326" velocity="2.5"/>
-      <dynamics D="1" K="7000" mu_coulomb="0" mu_viscous="16" damping="0.003" friction="0.0"/>
+      <!-- <dynamics D="1" K="7000" mu_coulomb="0" mu_viscous="16" damping="0.003" friction="0.0"/> -->
+      <dynamics D="1" K="7000" mu_coulomb="0" mu_viscous="16" damping="0.392" friction="0.992"/>
     </joint>
     <link name="${arm_id}_link3">
@@ -129,5 +131,6 @@
       <axis xyz="0 0 1"/>
       <limit acceleration="12.5" lower="-2.9671" effort="87" upper="2.9671" velocity="2.5"/>
-      <dynamics D="1" K="7000" mu_coulomb="0" mu_viscous="16" damping="0.003" friction="0.0"/>
+      <!-- <dynamics D="1" K="7000" mu_coulomb="0" mu_viscous="16" damping="0.003" friction="0.0"/> -->
+      <dynamics D="1" K="7000" mu_coulomb="0" mu_viscous="16" damping="0.457" friction="0.994"/>
     </joint>
     <link name="${arm_id}_link4">
@@ -159,5 +162,6 @@
       <axis xyz="0 0 1"/>
       <limit acceleration="12.5" lower="-3.1416" effort="87" upper="-0.4" velocity="2.5"/>
-      <dynamics D="1" K="7000" mu_coulomb="0" mu_viscous="16" damping="0.003" friction="0.0"/>
+      <!-- <dynamics D="1" K="7000" mu_coulomb="0" mu_viscous="16" damping="0.003" friction="0.0"/> -->
+      <dynamics D="1" K="7000" mu_coulomb="0" mu_viscous="16" damping="0.189" friction="0.677"/>
     </joint>
     <link name="${arm_id}_link5">
@@ -189,5 +193,6 @@
       <axis xyz="0 0 1"/>
       <limit acceleration="15" lower="-2.9671" effort="12" upper="2.9671" velocity="3"/>
-      <dynamics D="1" K="7000" mu_coulomb="0" mu_viscous="16" damping="0.003" friction="0.0"/>
+      <!-- <dynamics D="1" K="7000" mu_coulomb="0" mu_viscous="16" damping="0.003" friction="0.0"/> -->
+      <dynamics D="1" K="7000" mu_coulomb="0" mu_viscous="16" damping="0.077" friction="0.732"/>
     </joint>
     <link name="${arm_id}_link6">
@@ -220,5 +225,6 @@
       <axis xyz="0 0 1"/>
       <limit acceleration="20" lower="-0.0873" effort="12" upper="3.8223" velocity="3"/>
-      <dynamics D="1" K="7000" mu_coulomb="0" mu_viscous="16" damping="0.003" friction="0.0"/>
+      <!-- <dynamics D="1" K="7000" mu_coulomb="0" mu_viscous="16" damping="0.003" friction="0.0"/> -->
+      <dynamics D="1" K="7000" mu_coulomb="0" mu_viscous="16" damping="0.03" friction="0.428"/>
     </joint>
     <link name="${arm_id}_link7">
@@ -251,5 +257,6 @@
       <axis xyz="0 0 1"/>
       <limit acceleration="20" lower="-2.9671" effort="12" upper="2.9671" velocity="3"/>
-      <dynamics D="1" K="7000" mu_coulomb="0" mu_viscous="16" damping="0.003" friction="0.0"/>
+      <!-- <dynamics D="1" K="7000" mu_coulomb="0" mu_viscous="16" damping="0.003" friction="0.0"/> -->
+      <dynamics D="1" K="7000" mu_coulomb="0" mu_viscous="16" damping="0.06" friction="0.54"/>
     </joint>
     <link name="${arm_id}_link8" />

File: franka_description/robots/panda_real_env.xacro (robot description, xacro)
@@ -78,4 +78,15 @@
       <origin xyz="${panda_origin_to_table_centroid_offset} 0 -${board_height}"/>  <!-- -0.07450000000000001 z offset--> <!-- -0.05 + table_offset-->
     </joint>
+    <gazebo reference="table">
+      <mu1>0.35</mu1>
+      <mu2>0.35</mu2>
+      <collision>
+        <surface>
+          <contact>
+            <collide_bitmask>0x10</collide_bitmask>
+          </contact>
+        </surface>
+      </collision>
+    </gazebo>
   </xacro:macro>
 </robot>

Commit message: WIP merge of melodic contact estimation branch into noetic

File: franka_description/robots/panda_gazebo.xacro (robot description, xacro)
@@ -40,4 +40,5 @@
       </inertial>
     </link>
+    <xacro:gazebo-coll-bitmask link="${arm_id}_link0" bitmask="0x0" />
     <link name="${arm_id}_link1">
       <visual>
@@ -68,5 +69,6 @@
       <axis xyz="0 0 1"/>
       <limit acceleration="15" lower="-2.9671" effort="87" upper="2.9671" velocity="2.5"/>
-      <dynamics D="1" K="7000" mu_coulomb="0" mu_viscous="16" damping="0.003" friction="0.0"/>
+      <!-- <dynamics D="1" K="7000" mu_coulomb="0" mu_viscous="16" damping="0.003" friction="0.0"/> -->
+      <dynamics D="1" K="7000" mu_coulomb="0" mu_viscous="16" damping="0.32" friction="1.045"/>
     </joint>
     <link name="${arm_id}_link2">
@@ -98,5 +100,6 @@
       <axis xyz="0 0 1"/>
       <limit acceleration="7.5" lower="-1.8326" effort="87" upper="1.8326" velocity="2.5"/>
-      <dynamics D="1" K="7000" mu_coulomb="0" mu_viscous="16" damping="0.003" friction="0.0"/>
+      <!-- <dynamics D="1" K="7000" mu_coulomb="0" mu_viscous="16" damping="0.003" friction="0.0"/> -->
+      <dynamics D="1" K="7000" mu_coulomb="0" mu_viscous="16" damping="0.392" friction="0.992"/>
     </joint>
     <link name="${arm_id}_link3">
@@ -128,5 +131,6 @@
       <axis xyz="0 0 1"/>
       <limit acceleration="12.5" lower="-2.9671" effort="87" upper="2.9671" velocity="2.5"/>
-      <dynamics D="1" K="7000" mu_coulomb="0" mu_viscous="16" damping="0.003" friction="0.0"/>
+      <!-- <dynamics D="1" K="7000" mu_coulomb="0" mu_viscous="16" damping="0.003" friction="0.0"/> -->
+      <dynamics D="1" K="7000" mu_coulomb="0" mu_viscous="16" damping="0.457" friction="0.994"/>
     </joint>
     <link name="${arm_id}_link4">
@@ -158,5 +162,6 @@
       <axis xyz="0 0 1"/>
       <limit acceleration="12.5" lower="-3.1416" effort="87" upper="-0.4" velocity="2.5"/>
-      <dynamics D="1" K="7000" mu_coulomb="0" mu_viscous="16" damping="0.003" friction="0.0"/>
+      <!-- <dynamics D="1" K="7000" mu_coulomb="0" mu_viscous="16" damping="0.003" friction="0.0"/> -->
+      <dynamics D="1" K="7000" mu_coulomb="0" mu_viscous="16" damping="0.189" friction="0.677"/>
     </joint>
     <link name="${arm_id}_link5">
@@ -188,5 +193,6 @@
       <axis xyz="0 0 1"/>
       <limit acceleration="15" lower="-2.9671" effort="12" upper="2.9671" velocity="3"/>
-      <dynamics D="1" K="7000" mu_coulomb="0" mu_viscous="16" damping="0.003" friction="0.0"/>
+      <!-- <dynamics D="1" K="7000" mu_coulomb="0" mu_viscous="16" damping="0.003" friction="0.0"/> -->
+      <dynamics D="1" K="7000" mu_coulomb="0" mu_viscous="16" damping="0.077" friction="0.732"/>
     </joint>
     <link name="${arm_id}_link6">
@@ -211,4 +217,5 @@
       </inertial>
     </link>
+    <xacro:gazebo-coll-bitmask link="${arm_id}_link6" bitmask="0x01" />
     <joint name="${arm_id}_joint6" type="revolute">
       <safety_controller k_position="100.0" k_velocity="40.0" soft_lower_limit="-0.0175" soft_upper_limit="3.7525"/>
@@ -218,5 +225,6 @@
       <axis xyz="0 0 1"/>
       <limit acceleration="20" lower="-0.0873" effort="12" upper="3.8223" velocity="3"/>
-      <dynamics D="1" K="7000" mu_coulomb="0" mu_viscous="16" damping="0.003" friction="0.0"/>
+      <!-- <dynamics D="1" K="7000" mu_coulomb="0" mu_viscous="16" damping="0.003" friction="0.0"/> -->
+      <dynamics D="1" K="7000" mu_coulomb="0" mu_viscous="16" damping="0.03" friction="0.428"/>
     </joint>
     <link name="${arm_id}_link7">
@@ -241,4 +249,5 @@
       </inertial>
     </link>
+    <xacro:gazebo-coll-bitmask link="${arm_id}_link7" bitmask="0x01" />
     <joint name="${arm_id}_joint7" type="revolute">
       <safety_controller k_position="100.0" k_velocity="40.0" soft_lower_limit="-2.8973" soft_upper_limit="2.8973"/>
@@ -248,5 +257,6 @@
       <axis xyz="0 0 1"/>
       <limit acceleration="20" lower="-2.9671" effort="12" upper="2.9671" velocity="3"/>
-      <dynamics D="1" K="7000" mu_coulomb="0" mu_viscous="16" damping="0.003" friction="0.0"/>
+      <!-- <dynamics D="1" K="7000" mu_coulomb="0" mu_viscous="16" damping="0.003" friction="0.0"/> -->
+      <dynamics D="1" K="7000" mu_coulomb="0" mu_viscous="16" damping="0.06" friction="0.54"/>
     </joint>
     <link name="${arm_id}_link8" />
@@ -286,4 +296,5 @@
       </inertial>
     </link>
+    <xacro:gazebo-coll-bitmask link="${arm_id}_hand" bitmask="0x01" />
     <xacro:macro name="finger-collision" params="sign">
       <!-- screw mount -->
@@ -339,4 +350,6 @@
     <xacro:gazebo-friction link="${arm_id}_leftfinger" mu="1.13" />
     <xacro:gazebo-friction link="${arm_id}_rightfinger" mu="1.13" />
+    <xacro:gazebo-coll-bitmask link="${arm_id}_leftfinger" bitmask="0x01" />
+    <xacro:gazebo-coll-bitmask link="${arm_id}_rightfinger" bitmask="0x01" />
     <joint name="${arm_id}_finger_joint1" type="prismatic">
       <parent link="${arm_id}_hand"/>
@@ -357,3 +370,99 @@
     </joint>
   </xacro:macro>
+  <xacro:macro name="peg" params="connected_to:='' ns:='' xyz:='0 0 0' rpy:='0 0 0'">
+    <xacro:include filename="$(find franka_description)/robots/utils.xacro"/>
+    <xacro:unless value="${connected_to == ''}">
+      <joint name="${ns}_peg_joint" type="fixed">
+        <parent link="${connected_to}"/>
+        <child link="${ns}_peg"/>
+        <origin xyz="${xyz}" rpy="${rpy}"/>
+      </joint>
+    </xacro:unless>
+     <!-- 1" diameter and 4.375" length (including mount plate) -->
+    <xacro:property name="radius" value="0.0127" />
+    <xacro:property name="length" value="0.111125" />
+    <xacro:property name="mass" value="0.23" />
+    <link name="${ns}_peg">
+      <!-- <origin xyz="0 0 0" rpy="0 0 0"/> -->
+      <visual>
+        <origin xyz="0 0 ${length/2}" rpy="0 0 0"/>
+        <geometry>
+          <cylinder length="${length}" radius="${radius}"/>
+        </geometry>
+        <material name="gray">
+          <color rgba="0.75 0.75 0.75 1"/>
+        </material>
+      </visual>
+      <collision>
+        <origin xyz="0 0 ${length/2}" rpy="0 0 0"/>
+        <geometry>
+          <cylinder length="${length}" radius="${radius}"/>
+        </geometry>
+      </collision>
+      <inertial>
+        <origin xyz="0 0 ${length/2}"/>
+        <mass value="${mass}"/>
+      	<cylinder_inertia_def radius="${radius}" length="${length}" mass="${mass}"/>
+      </inertial>
+	  </link>
+    <gazebo reference="${ns}_peg">
+      <mu1>0.2</mu1>
+      <mu2>0.2</mu2>
+    </gazebo>
+    <!-- add a dummy link to the tip of the peg for rviz/kdl purposes -->
+    <joint name="${ns}_tip_joint" type="fixed">
+        <parent link="${ns}_peg"/>
+        <child link="${ns}_tip"/>
+        <origin xyz="0 0 0.111" rpy="0 0 0"/>
+    </joint>
+    <link name="${ns}_tip">
+    </link>
+  </xacro:macro>
+   <xacro:macro name="sphere_shape" params="connected_to:='' ns:='' rpy:='0 0 0' xyz:='0 0 0' radius:='' mu='' ">
+    <xacro:unless value="${connected_to == ''}">
+      <joint name="${ns}_sphere_joint" type="fixed">
+        <parent link="${connected_to}"/>
+        <child link="${ns}_sphere"/>
+        <origin xyz="${xyz}" rpy="${rpy}"/>
+      </joint>
+    </xacro:unless>
+    <xacro:property name="mass" value="0.23" />
+    <link name="${ns}_sphere">
+      <visual>
+        <origin xyz="0 0 ${radius}" rpy="0 0 0"/>
+        <geometry>
+          <sphere radius="${radius}"/>
+        </geometry>
+        <material name="gray">
+          <color rgba="0.75 0.75 0.75 1"/>
+        </material>
+      </visual>
+      <collision>
+        <origin xyz="0 0 ${radius}" rpy="0 0 0"/>
+        <geometry>
+          <sphere radius="${radius}"/>
+        </geometry>
+      </collision>
+      <inertial>
+        <origin xyz="0 0 ${radius}"/>
+        <mass value="${mass}"/>
+      	<sphere_inertia_def radius="${radius}" mass="${mass}"/>
+      </inertial>
+	  </link>
+    <gazebo reference="${ns}_sphere">
+      <mu1 value="${mu}" />
+      <mu2 value="${mu}" />
+      <!-- previously 1e5 -->
+      <kp>1e4</kp>
+      <kd>1e1</kd>
+    </gazebo>
+    <!-- add a dummy link to the tip of the peg for rviz/kdl purposes -->
+    <joint name="${ns}_tip_joint" type="fixed">
+        <parent link="${ns}_sphere"/>
+        <child link="${ns}_tip"/>
+        <origin xyz="0 0 ${radius * 2}" rpy="0 0 0"/>
+    </joint>
+    <link name="${ns}_tip">
+    </link>
+  </xacro:macro>
 </robot>
