Commit message: undo the simulated friction

File: franka_description/robots/panda_gazebo.xacro (robot description, xacro)
@@ -70,8 +70,6 @@
       <axis xyz="0 0 1"/>
       <limit acceleration="15" lower="-2.9671" effort="87" upper="2.9671" velocity="2.5"/>
-      <!-- <dynamics D="1" K="7000" mu_coulomb="0" mu_viscous="16" damping="0.003" friction="0.0"/> -->
-      <dynamics D="1" K="7000" mu_coulomb="0" mu_viscous="16" damping="0.32" friction="1.045"/>
-      <!-- <dynamics D="1" K="7000" mu_coulomb="0" mu_viscous="16" damping="0.003" friction="0.0"/> -->
-      <dynamics D="1" K="7000" mu_coulomb="0" mu_viscous="16" damping="0.32" friction="1.045"/>
+      <dynamics D="1" K="7000" mu_coulomb="0" mu_viscous="16" damping="0.003" friction="0.0"/>
+      <!-- <dynamics D="1" K="7000" mu_coulomb="0" mu_viscous="16" damping="0.32" friction="1.045"/> -->
     </joint>
     <link name="${arm_id}_link2">
@@ -103,8 +101,6 @@
       <axis xyz="0 0 1"/>
       <limit acceleration="7.5" lower="-1.8326" effort="87" upper="1.8326" velocity="2.5"/>
-      <!-- <dynamics D="1" K="7000" mu_coulomb="0" mu_viscous="16" damping="0.003" friction="0.0"/> -->
-      <dynamics D="1" K="7000" mu_coulomb="0" mu_viscous="16" damping="0.392" friction="0.992"/>
-      <!-- <dynamics D="1" K="7000" mu_coulomb="0" mu_viscous="16" damping="0.003" friction="0.0"/> -->
-      <dynamics D="1" K="7000" mu_coulomb="0" mu_viscous="16" damping="0.392" friction="0.992"/>
+      <dynamics D="1" K="7000" mu_coulomb="0" mu_viscous="16" damping="0.003" friction="0.0"/>
+      <!-- <dynamics D="1" K="7000" mu_coulomb="0" mu_viscous="16" damping="0.392" friction="0.992"/> -->
     </joint>
     <link name="${arm_id}_link3">
@@ -136,8 +132,6 @@
       <axis xyz="0 0 1"/>
       <limit acceleration="12.5" lower="-2.9671" effort="87" upper="2.9671" velocity="2.5"/>
-      <!-- <dynamics D="1" K="7000" mu_coulomb="0" mu_viscous="16" damping="0.003" friction="0.0"/> -->
-      <dynamics D="1" K="7000" mu_coulomb="0" mu_viscous="16" damping="0.457" friction="0.994"/>
-      <!-- <dynamics D="1" K="7000" mu_coulomb="0" mu_viscous="16" damping="0.003" friction="0.0"/> -->
-      <dynamics D="1" K="7000" mu_coulomb="0" mu_viscous="16" damping="0.457" friction="0.994"/>
+      <dynamics D="1" K="7000" mu_coulomb="0" mu_viscous="16" damping="0.003" friction="0.0"/>
+      <!-- <dynamics D="1" K="7000" mu_coulomb="0" mu_viscous="16" damping="0.457" friction="0.994"/> -->
     </joint>
     <link name="${arm_id}_link4">
@@ -169,8 +163,6 @@
       <axis xyz="0 0 1"/>
       <limit acceleration="12.5" lower="-3.1416" effort="87" upper="-0.4" velocity="2.5"/>
-      <!-- <dynamics D="1" K="7000" mu_coulomb="0" mu_viscous="16" damping="0.003" friction="0.0"/> -->
-      <dynamics D="1" K="7000" mu_coulomb="0" mu_viscous="16" damping="0.189" friction="0.677"/>
-      <!-- <dynamics D="1" K="7000" mu_coulomb="0" mu_viscous="16" damping="0.003" friction="0.0"/> -->
-      <dynamics D="1" K="7000" mu_coulomb="0" mu_viscous="16" damping="0.189" friction="0.677"/>
+      <dynamics D="1" K="7000" mu_coulomb="0" mu_viscous="16" damping="0.003" friction="0.0"/>
+      <!-- <dynamics D="1" K="7000" mu_coulomb="0" mu_viscous="16" damping="0.189" friction="0.677"/> -->
     </joint>
     <link name="${arm_id}_link5">
@@ -202,8 +194,6 @@
       <axis xyz="0 0 1"/>
       <limit acceleration="15" lower="-2.9671" effort="12" upper="2.9671" velocity="3"/>
-      <!-- <dynamics D="1" K="7000" mu_coulomb="0" mu_viscous="16" damping="0.003" friction="0.0"/> -->
-      <dynamics D="1" K="7000" mu_coulomb="0" mu_viscous="16" damping="0.077" friction="0.732"/>
-      <!-- <dynamics D="1" K="7000" mu_coulomb="0" mu_viscous="16" damping="0.003" friction="0.0"/> -->
-      <dynamics D="1" K="7000" mu_coulomb="0" mu_viscous="16" damping="0.077" friction="0.732"/>
+      <dynamics D="1" K="7000" mu_coulomb="0" mu_viscous="16" damping="0.003" friction="0.0"/>
+      <!-- <dynamics D="1" K="7000" mu_coulomb="0" mu_viscous="16" damping="0.077" friction="0.732"/> -->
     </joint>
     <link name="${arm_id}_link6">
@@ -236,8 +226,6 @@
       <axis xyz="0 0 1"/>
       <limit acceleration="20" lower="-0.0873" effort="12" upper="3.8223" velocity="3"/>
-      <!-- <dynamics D="1" K="7000" mu_coulomb="0" mu_viscous="16" damping="0.003" friction="0.0"/> -->
-      <dynamics D="1" K="7000" mu_coulomb="0" mu_viscous="16" damping="0.03" friction="0.428"/>
-      <!-- <dynamics D="1" K="7000" mu_coulomb="0" mu_viscous="16" damping="0.003" friction="0.0"/> -->
-      <dynamics D="1" K="7000" mu_coulomb="0" mu_viscous="16" damping="0.03" friction="0.428"/>
+      <dynamics D="1" K="7000" mu_coulomb="0" mu_viscous="16" damping="0.003" friction="0.0"/>
+      <!-- <dynamics D="1" K="7000" mu_coulomb="0" mu_viscous="16" damping="0.03" friction="0.428"/> -->
     </joint>
     <link name="${arm_id}_link7">
@@ -271,8 +259,6 @@
       <axis xyz="0 0 1"/>
       <limit acceleration="20" lower="-2.9671" effort="12" upper="2.9671" velocity="3"/>
-      <!-- <dynamics D="1" K="7000" mu_coulomb="0" mu_viscous="16" damping="0.003" friction="0.0"/> -->
-      <dynamics D="1" K="7000" mu_coulomb="0" mu_viscous="16" damping="0.06" friction="0.54"/>
-      <!-- <dynamics D="1" K="7000" mu_coulomb="0" mu_viscous="16" damping="0.003" friction="0.0"/> -->
-      <dynamics D="1" K="7000" mu_coulomb="0" mu_viscous="16" damping="0.06" friction="0.54"/>
+      <dynamics D="1" K="7000" mu_coulomb="0" mu_viscous="16" damping="0.003" friction="0.0"/>
+      <!-- <dynamics D="1" K="7000" mu_coulomb="0" mu_viscous="16" damping="0.06" friction="0.54"/> -->
     </joint>
     <link name="${arm_id}_link8" />
