Commit message: add texture to tabletop

File: franka_description/robots/tabletop.xacro (robot description, xacro)
@@ -64,4 +64,5 @@
           <box size="${table_length} ${table_width} ${table_height}"/>
         </geometry>
+        <!-- add a texture -->
       </visual>
       <collision>
@@ -88,4 +89,16 @@
         </surface>
       </collision>
+      <material>Gazebo/DarkGrey</material>
+    </gazebo>
+    <gazebo reference="mount_plate">
+      <material>Gazebo/DarkGrey</material>
+      <!-- <visual>
+        <material>
+          <ambient>0.5 0.0 0.0 1</ambient>
+          <diffuse>0.5 0.0 0.0 1</diffuse>
+          <specular>0 0 0 0</specular>
+          <emissive>0 0 0 1</emissive>
+        </material>
+      </visual> -->
     </gazebo>
   </xacro:macro>
