Commit message: add radius and friction param

File: franka_description/robots/panda_arm_attachments.urdf.xacro (robot description, xacro)
@@ -4,6 +4,8 @@
   <xacro:arg name="hand"   default="false" /> <!-- Should a franka_gripper be mounted at the flange?" -->
   <xacro:arg name="gazebo" default="false" /> <!-- Is the robot being simulated in gazebo?" -->
-  <xacro:arg name="peg"    default="false"/> <!-- Should a peg be mounted at the flange?" -->
+  <xacro:arg name="peg"    default="false" /> <!-- Should a peg be mounted at the flange?" -->
   <xacro:arg name="sphere" default="false" /> <!-- Should a sphere be mounted at the flange? -->
+  <xacro:arg name="radius" default="1.0"   /> <!-- How large should the sphere be in [m]? -->
+  <xacro:arg name="mu"     default="0.2"   /> <!-- What is the coefficient of friction? -->
   <xacro:property name="arm_id" value="$(arg arm_id)" />
   <!-- Create a URDF for a real hardware -->
@@ -21,5 +23,5 @@
     <xacro:if value="$(arg sphere)">
       <xacro:include filename="$(find franka_description)/robots/sphere.xacro"/>
-      <xacro:sphere_shape ns="${arm_id}" rpy="0 0 ${-pi/4}" connected_to="${arm_id}_link8"/>
+      <xacro:sphere_shape ns="${arm_id}" rpy="0 0 ${-pi/4}" connected_to="${arm_id}_link8" radius="$(arg radius) mu=$(arg mu) "/>
     </xacro:if>
   </xacro:unless>
@@ -41,5 +43,5 @@
     </xacro:if>
     <xacro:if value="$(arg sphere)">
-      <xacro:sphere_shape ns="${arm_id}" rpy="0 0 ${-pi/4}" connected_to="${arm_id}_link8" />
+      <xacro:sphere_shape ns="${arm_id}" rpy="0 0 ${-pi/4}" connected_to="${arm_id}_link8" radius="$(arg radius)" mu="$(arg mu)" />
     </xacro:if>
     <!-- Gazebo requires a joint to a link called "world" for statically mounted robots -->

File: franka_description/robots/panda_gazebo.xacro (robot description, xacro)
@@ -407,5 +407,5 @@
     </link>
   </xacro:macro>
-   <xacro:macro name="sphere_shape" params="connected_to:='' ns:='' rpy:='0 0 0' xyz:='0 0 0' ">
+   <xacro:macro name="sphere_shape" params="connected_to:='' ns:='' rpy:='0 0 0' xyz:='0 0 0' radius:='' mu='' ">
     <xacro:unless value="${connected_to == ''}">
       <joint name="${ns}_sphere_joint" type="fixed">
@@ -415,5 +415,4 @@
       </joint>
     </xacro:unless>
-    <xacro:property name="radius" value="0.0555625" />
     <xacro:property name="mass" value="0.23" />
     <link name="${ns}_sphere">
@@ -440,6 +439,6 @@
 	  </link>
     <gazebo reference="${ns}_sphere">
-      <mu1>0.2</mu1>
-      <mu2>0.2</mu2>
+      <mu1 value="${mu}" />
+      <mu2 value="${mu}" />
     </gazebo>
     <!-- add a dummy link to the tip of the peg for rviz/kdl purposes -->

File: franka_description/robots/sphere.xacro (robot description, xacro)
@@ -3,5 +3,5 @@
   <!-- utils /-->
   <xacro:include filename="$(find franka_description)/robots/utils.xacro"/>
-  <xacro:macro name="sphere_shape" params="connected_to:='' ns:='' rpy:='0 0 0' xyz:='0 0 0' ">
+  <xacro:macro name="sphere_shape" params="connected_to:='' ns:='' rpy:='0 0 0' xyz:='0 0 0' radius='' ">
     <xacro:unless value="${connected_to == ''}">
       <joint name="${ns}_sphere_joint" type="fixed">
@@ -11,5 +11,5 @@
       </joint>
     </xacro:unless>
-    <xacro:property name="radius" value="0.0555625" />
+    <xacro:property name="radius" value="${radius}" />
     <xacro:property name="mass" value="0.23" />
     <link name="${ns}_sphere">
@@ -35,9 +35,9 @@
       </inertial>
 	  </link>
-    <!-- add a dummy link to the tip of the peg for rviz/kdl purposes -->
+    <!-- add a dummy link to the tip of the sphere for rviz/kdl purposes -->
     <joint name="${ns}_tip_joint" type="fixed">
         <parent link="${ns}_sphere"/>
         <child link="${ns}_tip"/>
-        <origin xyz="0 0 0.555" rpy="0 0 0"/>
+        <origin xyz="0 0 ${radius}" rpy="0 0 0"/>
     </joint>
     <link name="${ns}_tip">

Commit message: correct xacro file

File: franka_description/robots/panda_arm_attachments.urdf.xacro (robot description, xacro)
@@ -1,23 +1,24 @@
 <?xml version='1.0' encoding='utf-8'?>
 <robot xmlns:xacro="http://www.ros.org/wiki/xacro" name="panda">
-  <xacro:arg name="arm_id"       default="panda" /> <!-- Name of this panda -->
-  <xacro:arg name="end_effector" default=""      /> <!-- What should be mounted at the flange [hand, peg, sphere]? -->
-  <xacro:arg name="gazebo"       default="false" /> <!-- Is the robot being simulated in gazebo?" -->
-  <xacro:arg name="radius"       default="1.0"   /> <!-- How large should the sphere be in [m]? -->
-  <xacro:arg name="mu"           default="0.2"   /> <!-- What is the coefficient of friction? -->
-  <xacro:property name="arm_id" value="$(arg arm_id)" />
+  <xacro:arg      name="arm_id"       default="panda" /> <!-- Name of this panda -->
+  <xacro:arg      name="end_effector" default=""      /> <!-- What should be mounted at the flange [hand, peg, sphere]? -->
+  <xacro:arg      name="gazebo"       default="false" /> <!-- Is the robot being simulated in gazebo?" -->
+  <xacro:arg      name="radius"       default="1.0"   /> <!-- How large should the sphere be in [m]? -->
+  <xacro:arg      name="mu"           default="0.2"   /> <!-- What is the coefficient of friction? -->
+  <xacro:property name="arm_id"       value="$(arg arm_id)" />
+  <xacro:property name="end_effector"   value="$(arg end_effector)" />
   <!-- Create a URDF for a real hardware -->
   <xacro:unless value="$(arg gazebo)">
     <xacro:include filename="$(find franka_description)/robots/panda_arm.xacro" />
     <xacro:panda_arm arm_id="${arm_id}" safety_distance="0.03"/>
-    <xacro:if value="$(arg end_effector == hand)">
+    <xacro:if value="${end_effector == 'hand'}">
       <xacro:include filename="$(find franka_description)/robots/hand.xacro"/>
       <xacro:hand ns="${arm_id}" rpy="0 0 ${-pi/4}" connected_to="${arm_id}_link8" safety_distance="0.03"/>
     </xacro:if>
-    <xacro:if value="$(arg end_effector == peg)">
+    <xacro:if value="${end_effector == 'peg'}">
       <xacro:include filename="$(find franka_description)/robots/peg.xacro"/>
       <xacro:peg ns="${arm_id}" rpy="0 0 ${-pi/4}" connected_to="${arm_id}_link8"/>
     </xacro:if>
-    <xacro:if value="$(arg end_effector == sphere)">
+    <xacro:if value="${end_effector == 'sphere'}">
       <xacro:include filename="$(find franka_description)/robots/sphere.xacro"/>
       <xacro:sphere_shape ns="${arm_id}" rpy="0 0 ${-pi/4}" connected_to="${arm_id}_link8" radius="$(arg radius) mu=$(arg mu) "/>
@@ -32,13 +33,14 @@
     <xacro:include filename="$(find franka_description)/robots/panda_gazebo.xacro" />
     <xacro:panda_arm arm_id="${arm_id}" />
-    <xacro:if value="$(arg end_effector == hand)">
+    <xacro:if value="${end_effector == 'hand'}">
       <xacro:hand ns="${arm_id}" rpy="0 0 ${-pi/4}" connected_to="${arm_id}_link8" />
       <xacro:gazebo-joint joint="${arm_id}_finger_joint1" transmission="hardware_interface/EffortJointInterface" />
       <xacro:gazebo-joint joint="${arm_id}_finger_joint2" transmission="hardware_interface/EffortJointInterface" />
     </xacro:if>
-    <xacro:if value="$(arg end_effector == peg)">
+    <xacro:if value="${end_effector == 'peg'}">
       <xacro:peg ns="${arm_id}" rpy="0 0 ${-pi/4}" connected_to="${arm_id}_link8" />
     </xacro:if>
-    <xacro:if value="$(arg end_effector == sphere)">
+]
+    <xacro:if value="${end_effector == 'sphere'}">
       <xacro:sphere_shape ns="${arm_id}" rpy="0 0 ${-pi/4}" connected_to="${arm_id}_link8" radius="$(arg radius)" mu="$(arg mu)" />
     </xacro:if>

Commit message: add real hw environment objects (table and lumped mounting board)

File: franka_description/robots/panda_arm_attachments.urdf.xacro (robot description, xacro)
@@ -6,6 +6,8 @@
   <xacro:arg      name="radius"       default="1.0"   /> <!-- How large should the sphere be in [m]? -->
   <xacro:arg      name="mu"           default="0.2"   /> <!-- What is the coefficient of friction? -->
+  <xacro:arg      name="real_env"           default="false"   /> <!-- What is the coefficient of friction? -->
   <xacro:property name="arm_id"       value="$(arg arm_id)" />
   <xacro:property name="end_effector"   value="$(arg end_effector)" />
+  <xacro:property name="real_env"   value="$(arg real_env)" />
   <!-- Create a URDF for a real hardware -->
   <xacro:unless value="$(arg gazebo)">
@@ -30,7 +32,11 @@
     <xacro:arg name="rpy" default="0 0 0" />
     <!-- Create a simulatable URDF -->
+    <xacro:include filename="$(find franka_description)/robots/panda_gazebo.xacro" />
     <xacro:include filename="$(find franka_description)/robots/utils.xacro" />
-    <xacro:include filename="$(find franka_description)/robots/panda_gazebo.xacro" />
+    <xacro:include filename="$(find franka_description)/robots/panda_real_env.xacro" />
     <xacro:panda_arm arm_id="${arm_id}" />
+    <xacro:if value="$(arg real_env)">
+        <xacro:environment/>
+    </xacro:if>
     <xacro:if value="${end_effector == 'hand'}">
       <xacro:hand ns="${arm_id}" rpy="0 0 ${-pi/4}" connected_to="${arm_id}_link8" />

Commit message: WIP get everything running on noetic again

File: franka_description/robots/panda_arm_attachments.urdf.xacro (robot description, xacro)
@@ -6,8 +6,8 @@
   <xacro:arg      name="radius"       default="1.0"   /> <!-- How large should the sphere be in [m]? -->
   <xacro:arg      name="mu"           default="0.2"   /> <!-- What is the coefficient of friction? -->
-  <xacro:arg      name="real_env"           default="false"   /> <!-- What is the coefficient of friction? -->
+  <xacro:arg      name="tabletop"           default="false"   /> <!-- What is the coefficient of friction? -->
   <xacro:property name="arm_id"       value="$(arg arm_id)" />
   <xacro:property name="end_effector"   value="$(arg end_effector)" />
-  <xacro:property name="real_env"   value="$(arg real_env)" />
+  <xacro:property name="tabletop"   value="$(arg tabletop)" />
   <!-- Create a URDF for a real hardware -->
   <xacro:unless value="$(arg gazebo)">
@@ -34,8 +34,8 @@
     <xacro:include filename="$(find franka_description)/robots/panda_gazebo.xacro" />
     <xacro:include filename="$(find franka_description)/robots/utils.xacro" />
-    <xacro:include filename="$(find franka_description)/robots/panda_real_env.xacro" />
+    <xacro:include filename="$(find franka_description)/robots/tabletop.xacro" />
     <xacro:panda_arm arm_id="${arm_id}" />
-    <xacro:if value="$(arg real_env)">
-        <xacro:environment/>
+    <xacro:if value="$(arg tabletop)">
+        <xacro:tabletop/>
     </xacro:if>
     <xacro:if value="${end_effector == 'hand'}">

Commit message: add texture files to backdrop and table

File: franka_description/robots/panda_arm_attachments.urdf.xacro (robot description, xacro)
@@ -7,4 +7,5 @@
   <xacro:arg      name="mu"           default="0.2"   /> <!-- What is the coefficient of friction? -->
   <xacro:arg      name="tabletop"           default="false"   /> <!-- What is the coefficient of friction? -->
+  <xacro:arg      name="backdrop"           default="false"   /> <!-- What is the coefficient of friction? -->
   <xacro:property name="arm_id"       value="$(arg arm_id)" />
   <xacro:property name="end_effector"   value="$(arg end_effector)" />
@@ -38,4 +39,7 @@
     <xacro:if value="$(arg tabletop)">
         <xacro:tabletop/>
+    </xacro:if>
+    <xacro:if value="$(arg backdrop)">
+        <xacro:backdrop/>
     </xacro:if>
     <xacro:if value="${end_effector == 'hand'}">

File: franka_description/robots/tabletop.xacro (robot description, xacro)
@@ -89,8 +89,22 @@
         </surface>
       </collision>
-      <material>Gazebo/DarkGrey</material>
+      <material>Franka/Random2</material>
+      <!-- <material>
+        <script>
+          <uri>model://franka/materials/scripts/</uri>
+          <uri>model://franka/materials/textures/</uri>
+          <name>Franka/Random1</name>
+        </script>
+      </material> -->
     </gazebo>
     <gazebo reference="mount_plate">
-      <material>Gazebo/DarkGrey</material>
+      <!-- <material>
+        <script>
+          <uri>model://franka/materials/scripts/</uri>
+          <uri>model://franka/materials/textures/</uri>
+          <name>Franka/Random2</name>
+        </script>
+      </material> -->
+      <material>Franka/Random2</material>
       <!-- <visual>
         <material>
@@ -103,3 +117,51 @@
     </gazebo>
   </xacro:macro>
+  <xacro:property name="wall_length" value="2" />
+  <xacro:property name="wall_width" value="4" />
+  <xacro:property name="wall_height" value="0.1" />
+  <xacro:property name="base_to_back_wall" value="1" />
+  <xacro:macro name="backdrop" params="">
+    <link name="back_wall">
+      <gazebo>
+		    <static>true</static>
+	    </gazebo>
+      <visual>
+        <origin xyz="0 0 -${wall_height/2}" />
+        <geometry>
+          <box size="${wall_length} ${wall_width} ${wall_height}"/>
+        </geometry>
+      </visual>
+      <collision>
+        <origin xyz="0 0 -${wall_height/2}" />
+        <geometry>
+          <box size="${wall_length} ${wall_width} ${wall_height}"/>
+        </geometry>
+      </collision>
+      <inertial>
+        <origin xyz="0 0 -${wall_height/2}" />
+        <mass value="1"/>
+        <!-- Inertia values were calculated to be consistent with the mass and
+            geometry size, assuming a uniform density. -->
+        <inertia ixx="100"  ixy="0"  ixz="0" iyy="100" iyz="0" izz="100" />
+      </inertial>
+    </link>
+    <joint name="base_to_back_wall" type="fixed">
+      <parent link="panda_link0"/>
+      <child link="back_wall"/>
+      <origin xyz="-${base_to_back_wall} 0 0" rpy="0 1.57079632679 0"/>
+    </joint>
+    <gazebo reference="back_wall">
+      <mu1>0.35</mu1>
+      <mu2>0.35</mu2>
+      <collision>
+        <surface>
+          <contact>
+            <collide_bitmask>0x10</collide_bitmask>
+          </contact>
+        </surface>
+      </collision>
+      <!-- <material>Gazebo/CloudySky</material> -->
+      <material>Franka/Random1</material>
+    </gazebo>
+  </xacro:macro>
 </robot>
